Commit message: rebuilding autonomous nav

File: urdf/base.xacro (robot description, xacro)
@@ -168,5 +168,5 @@
       <origin xyz="0 0 0" rpy="0 0 ${cad_yaw}"/>
       <geometry>
-        <mesh filename="package://zeko_description/meshes/base_link.stl" scale="0.001 0.001 0.001"/>
+        <mesh filename="package://robot_base_simulation/meshes/base_link.stl" scale="0.001 0.001 0.001"/>
       </geometry>
       <material name="zeko_chassis_grey"/>

File: urdf/casters.xacro (robot description, xacro)
@@ -26,5 +26,5 @@
         <origin xyz="${-x_sign * caster_x_offset} 0 ${-caster_radius}" rpy="0 0 ${cad_yaw}"/>
         <geometry>
-          <mesh filename="package://zeko_description/meshes/${prefix}_caster_fork.stl" scale="0.001 0.001 0.001"/>
+          <mesh filename="package://robot_base_simulation/meshes/${prefix}_caster_fork.stl" scale="0.001 0.001 0.001"/>
         </geometry>
         <material name="zeko_caster_dark_grey"/>
@@ -33,5 +33,5 @@
         <origin xyz="${-x_sign * caster_x_offset} 0 ${-caster_radius}" rpy="0 0 ${cad_yaw}"/>
         <geometry>
-          <mesh filename="package://zeko_description/meshes/${prefix}_caster_wheel.stl" scale="0.001 0.001 0.001"/>
+          <mesh filename="package://robot_base_simulation/meshes/${prefix}_caster_wheel.stl" scale="0.001 0.001 0.001"/>
         </geometry>
         <material name="zeko_wheel_black"/>

File: urdf/pelvis_mount.xacro (robot description, xacro)
@@ -20,5 +20,5 @@
       <origin xyz="0 0 -0.504" rpy="0 0 ${cad_yaw}"/>
       <geometry>
-        <mesh filename="package://zeko_description/meshes/pelvis_mount_link.stl" scale="0.001 0.001 0.001"/>
+        <mesh filename="package://robot_base_simulation/meshes/pelvis_mount_link.stl" scale="0.001 0.001 0.001"/>
       </geometry>
       <material name="zeko_pelvis_blue"/>

File: urdf/support_frame.xacro (robot description, xacro)
@@ -19,5 +19,5 @@
       <origin xyz="0 0 -0.221" rpy="0 0 ${cad_yaw}"/>
       <geometry>
-        <mesh filename="package://zeko_description/meshes/support_frame_link.stl" scale="0.001 0.001 0.001"/>
+        <mesh filename="package://robot_base_simulation/meshes/support_frame_link.stl" scale="0.001 0.001 0.001"/>
       </geometry>
       <material name="zeko_frame_silver"/>

File: urdf/wheels.xacro (robot description, xacro)
@@ -31,5 +31,5 @@
         <origin xyz="0 ${-reflect * wheel_separation / 2.0} ${-wheel_radius}" rpy="0 0 ${cad_yaw}"/>
         <geometry>
-          <mesh filename="package://zeko_description/meshes/${prefix}_wheel_link.stl" scale="0.001 0.001 0.001"/>
+          <mesh filename="package://robot_base_simulation/meshes/${prefix}_wheel_link.stl" scale="0.001 0.001 0.001"/>
         </geometry>
         <material name="zeko_wheel_black"/>

File: urdf/zeko.urdf (robot description, URDF)
Before this commit: robot zeko, 7 links, 6 joints
Links:
- added link body_link; visual mesh filename=package://robot_base_simulation/meshes/zeko_body.obj scale=0.01 0.01 0.01
- added link lidar_link, mass 0.001; visual cylinder length=0.06 radius=0.05
- link base_link: geometry collision box size=1.0 0.65 0.124; visual mesh filename=package://robot_base_simulation/meshes/base_link.stl scale=0.001 0.001 0.001
- link front_caster_link: geometry collision sphere radius=0.045; visual mesh filename=package://robot_base_simulation/meshes/front_caster_fork.stl scale=0.001 0.001 0.001
- link left_wheel_link: geometry collision cylinder length=0.08 radius=0.1524; visual mesh filename=package://robot_base_simulation/meshes/left_wheel_link.stl scale=0.001 0.001 0.001
- link pelvis_mount_link: geometry collision box size=0.225 0.285 0.152; visual mesh filename=package://robot_base_simulation/meshes/pelvis_mount_link.stl scale=0.001 0.001 0.001
- link rear_caster_link: geometry collision sphere radius=0.045; visual mesh filename=package://robot_base_simulation/meshes/rear_caster_fork.stl scale=0.001 0.001 0.001
- link right_wheel_link: geometry collision cylinder length=0.08 radius=0.1524; visual mesh filename=package://robot_base_simulation/meshes/right_wheel_link.stl scale=0.001 0.001 0.001
- link support_frame_link: geometry collision box size=0.348 0.268 0.283; visual mesh filename=package://robot_base_simulation/meshes/support_frame_link.s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 scale=0.001 0.001 0.001
Joints:
- added joint body_joint: type fixed, parent pelvis_mount_link, child body_link, origin xyz=0 0 0.152 rpy=0 0 0
- added joint lidar_joint: type fixed, parent base_link, child lidar_link, origin xyz=0.0 0.0 0.68 rpy=0 0 0.0

File: urdf/zeko.xacro (robot description, xacro)
@@ -25,10 +25,10 @@
        xacro:property values and inertia macros used by every other
        module below. -->
-  <xacro:include filename="$(find zeko_description)/urdf/materials.xacro"/>
-  <xacro:include filename="$(find zeko_description)/urdf/base.xacro"/>
-  <xacro:include filename="$(find zeko_description)/urdf/wheels.xacro"/>
-  <xacro:include filename="$(find zeko_description)/urdf/casters.xacro"/>
-  <xacro:include filename="$(find zeko_description)/urdf/support_frame.xacro"/>
-  <xacro:include filename="$(find zeko_description)/urdf/pelvis_mount.xacro"/>
+  <xacro:include filename="$(find robot_base_simulation)/urdf/materials.xacro"/>
+  <xacro:include filename="$(find robot_base_simulation)/urdf/base.xacro"/>
+  <xacro:include filename="$(find robot_base_simulation)/urdf/wheels.xacro"/>
+  <xacro:include filename="$(find robot_base_simulation)/urdf/casters.xacro"/>
+  <xacro:include filename="$(find robot_base_simulation)/urdf/support_frame.xacro"/>
+  <xacro:include filename="$(find robot_base_simulation)/urdf/pelvis_mount.xacro"/>
   <!-- =====================================================================
        ros2_control HARDWARE INTERFACE
